Commit message: added camera plugins on bot

File: go1_sim/go1_description/xacro/robot.xacro (robot description, xacro)
@@ -89,4 +89,56 @@
     <xacro:leg name="RR" mirror="-1" mirror_dae="False"  front_hind="-1" front_hind_dae="False" />
     <xacro:leg name="RL" mirror="1"  mirror_dae="True"   front_hind="-1" front_hind_dae="False" />
+     <!-- Camera joint and link (mounted at the front of the trunk) -->
+    <joint name="head_camera_joint" type="fixed">
+        <parent link="trunk"/>
+        <child link="head_camera_link"/>
+        <origin xyz="0.28 0 0.02" rpy="0 0 0"/>
+    </joint>
+    <link name="head_camera_link">
+        <visual>
+            <origin xyz="0 0 0" rpy="0 0 0"/>
+            <geometry>
+                <box size="0.03 0.03 0.03"/>
+            </geometry>
+            <material name="black"/>
+        </visual>
+        <collision>
+            <origin xyz="0 0 0" rpy="0 0 0"/>
+            <geometry>
+                <box size="0.03 0.03 0.03"/>
+            </geometry>
+        </collision>
+        <inertial>
+            <mass value="0.01"/>
+            <origin xyz="0 0 0" rpy="0 0 0"/>
+            <inertia ixx="1e-5" ixy="0" ixz="0" iyy="1e-5" iyz="0" izz="1e-5"/>
+        </inertial>
+    </link>
+    <gazebo reference="head_camera_link">
+        <sensor type="camera" name="head_camera">
+            <pose>0 0 0 0 0 0</pose>
+            <visualize>true</visualize>
+            <update_rate>30</update_rate>
+            <camera>
+                <horizontal_fov>1.3962634</horizontal_fov>
+                <image>
+                    <width>640</width>
+                    <height>480</height>
+                    <format>R8G8B8</format>
+                </image>
+                <clip>
+                    <near>0.02</near>
+                    <far>50</far>
+                </clip>
+            </camera>
+            <plugin name="camera_controller" filename="libgazebo_ros_camera.so">
+                <ros>
+                    <remapping>~/image_raw:=head_camera/image_raw</remapping>
+                </ros>
+                <camera_name>head_camera</camera_name>
+                <frame_name>head_camera_link</frame_name>
+            </plugin>
+        </sensor>
+    </gazebo>
     <!-- <xacro:depthCamera camID="1" name="face">
         <origin rpy="0 0 0" xyz="0.2785 -0.0125 0.0167"/>
@@ -103,5 +155,5 @@
     <xacro:depthCamera camID="5" name="rearDown">
         <origin rpy="0 ${PI/2} 0" xyz="-0.0825 -0.0125 -0.04365"/>
-    </xacro:depthCamera> -->
+    </xacro:depthCamera>  -->
     <!-- <joint name="camera_laserscan_joint_left" type="fixed">
         <origin rpy="0 0.2618 0" xyz="0 0 0"/>
